Commit message: paolo: update for integration with unipd - update launcher for using our abb

File: abb_description/urdf/irb6700_205_280_macro.xacro (robot description, xacro)
@@ -8,4 +8,5 @@
   <color rgba=".7 .7 .7 1"/>
 </material>
+<link name="world"/>
 <link name="${prefix}fake_linear_axis"/>
 <link name="${prefix}base_link">
@@ -122,4 +123,9 @@
 </link>
 <!--  joint list -->
+<joint name="${prefix}joint_world" type="fixed">
+  <origin xyz="-8 1 0" rpy="0 0 0"/>
+  <parent link="world"/>
+  <child link="${prefix}fake_linear_axis"/>
+</joint>
 <joint name="${prefix}joint_0" type="prismatic">
   <origin xyz="0 0 0" rpy="0 0 0"/>
