Commit message: paolo:config updates

File: abb_description/urdf/irb6700_205_280.xacro (robot description, xacro)
@@ -2,3 +2,30 @@
   <xacro:include filename="$(find abb_description)/urdf/irb6700_205_280_macro.xacro"/>
   <xacro:abb_irb6700_205_280 prefix=""/>
+  <joint name="$joint_ee" type="fixed">
+    <origin xyz="0.51 0 0" rpy="0 0 0"/>
+    <parent link="link_6"/>
+    <child link="gripper"/>
+  </joint>
+   <link name="gripper">
+   <inertial>
+     <origin xyz="0 0 0" rpy="0 0 0"/>
+     <mass value="1"/>
+     <inertia ixx="100"  ixy="0"  ixz="0" iyy="100" iyz="0" izz="100" />
+   </inertial>
+   <visual>
+     <origin xyz="0 0 0" rpy="0 0 0" />
+     <geometry>
+       <box size="1 1.7 .9" />
+     </geometry>
+     <material name="Cyan">
+       <color rgba="0 1.0 1.0 1.0"/>
+     </material>
+   </visual>
+   <collision>
+     <origin xyz="0 0 0" rpy="0 0 0"/>
+     <geometry>
+       <box size="1 1.7 .9" />
+     </geometry>
+   </collision>
+ </link>
 </robot>

Commit message: paolo: use prof pc

File: abb_description/urdf/irb6700_205_280.xacro (robot description, xacro)
@@ -29,3 +29,9 @@
    </collision>
  </link>
+   <joint name="$joint_deformation" type="fixed">
+    <origin xyz="1 0.85 0" rpy="0 1.5707 0"/>
+    <parent link="link_6"/>
+    <child link="grasping"/>
+  </joint>
+   <link name="grasping"/>
 </robot>

File: abb_description/urdf/irb6700_205_280_macro.xacro (robot description, xacro)
@@ -127,5 +127,5 @@
   <child link="${prefix}base_link"/>
   <axis xyz="0 0 1"/>
-  <limit lower="0" upper="0" effort="0" velocity="1"/>
+  <limit lower="-0.001" upper="0" effort="0" velocity="1"/>
 </joint>
 <joint name="${prefix}joint_1" type="revolute">

Commit message: paolo: parameters tuning / launcher

File: abb_description/urdf/irb6700_205_280.xacro (robot description, xacro)
@@ -16,5 +16,6 @@
      <origin xyz="0 0 0" rpy="0 0 0" />
      <geometry>
-       <box size="1 1.7 .9" />
+       <box size=".1 .1 .1" />
+       <!--box size="1 1.7 .9" /-->
      </geometry>
      <material name="Cyan">
@@ -30,5 +31,5 @@
  </link>
    <joint name="$joint_deformation" type="fixed">
-    <origin xyz="1 0.85 0" rpy="0 1.5707 0"/>
+    <origin xyz="0.78 0.86 -0.18" rpy="0 1.5707 0"/>
     <parent link="link_6"/>
     <child link="grasping"/>

Commit message: paolo: pforactr july

File: abb_description/urdf/irb6700_205_280.xacro (robot description, xacro)
@@ -16,9 +16,9 @@
      <origin xyz="0 0 0" rpy="0 0 0" />
      <geometry>
-       <box size=".1 .1 .1" />
-       <!--box size="1 1.7 .9" /-->
+       <!--box size=".1 .1 .1" /-->
+       <box size="1 1.7 .9" />
      </geometry>
      <material name="Cyan">
-       <color rgba="0 1.0 1.0 1.0"/>
+       <color rgba="0 1.0 1.0 0.5"/>
      </material>
    </visual>
@@ -31,5 +31,5 @@
  </link>
    <joint name="$joint_deformation" type="fixed">
-    <origin xyz="0.78 0.86 -0.18" rpy="0 1.5707 0"/>
+    <origin xyz="0.78 0.96 -0.18" rpy="0 1.5707 0"/>
     <parent link="link_6"/>
     <child link="grasping"/>

Commit message: minor changes on Dallara setup

File: abb_description/urdf/irb6700_205_280.xacro (robot description, xacro)
@@ -31,5 +31,5 @@
  </link>
    <joint name="$joint_deformation" type="fixed">
-    <origin xyz="0.78 0.96 -0.18" rpy="0 1.5707 0"/>
+    <origin xyz="0.78 0.744 0" rpy="0 1.5707 0"/>
     <parent link="link_6"/>
     <child link="grasping"/>
